File: eagle/daq.brd (EAGLE design)
At the start: 59.7 x 65.4 mm, 77 parts

Commit message: do
Parts:
- added R29: (no value), myparts:0805
- added R30, R31, R32: (no value), myparts:0603
- R19: device myparts:1206 -> myparts:0805
- R21, R22, R26, R28: device myparts:0603 -> myparts:0805
- R24: device myparts:1206 -> myparts:0603
- moved R24 21.8 mm to (41.1, 31.0), turned to 0 degrees
- moved R22 17.6 mm to (35.7, 11.0)
- moved R23 17.6 mm to (33.1, 22.6)
- moved R28 13.2 mm to (47.0, 11.0)
- moved R27 10.5 mm to (43.7, 14.6), turned to 0 degrees
- moved R21 10.4 mm to (39.2, 11.0)
- moved R26 7.78 mm to (45.2, 13.0), turned to 0 degrees
- moved R25 4.40 mm to (46.7, 14.6), turned to 180 degrees
- moved R19 3.43 mm to (37.5, 13.0)
- moved C15 3.18 mm to (19.8, 42.5)
- moved C16 3.18 mm to (35.6, 45.2)
- moved C2 3.18 mm to (41.1, 35.6)
- moved C5 3.18 mm to (32.0, 45.2)
- moved CON1 3.18 mm to (24.4, 35.6)
- moved IC1 3.18 mm to (34.3, 38.9)
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Connections:
- new net N$11: R18.2, R19.2, R21.2
- new net N$28: CON5.9, R29.1
- new net N$29: CON5.10, R28.1
- new net N$5: R19.1, R20.2, R22.2
- net N$15: now also R24.2; no longer R22.2
- net N$17: now also R27.2; no longer R25.2
- net N$21: now also R25.2; no longer R23.2
- net N$27: now also R30.2; no longer R26.2
- net N$40: now also R25.1, R26.2, R28.2; no longer CON5.10, R23.1, R24.1
- net N$59: now also R22.1; no longer R19.1, R20.2
- net N$71: now also R23.2; no longer R21.2
- net N$73: now also R32.2; no longer R28.2
- net N$79: now also R31.2; no longer R27.2
- net N$8: now also R26.1, R27.1, R29.2; no longer CON5.9, R24.2, R25.1
- net N$81: now also R21.1; no longer R18.2, R19.2
- net VCC: now also R23.1, R24.1, R30.1, R31.1, R32.1; no longer R21.1, R22.1, R26.1, R27.1, R28.1
Routing:
- net N$29: track 0.00 -> 4.94 mm
- net N$28: track 0.00 -> 4.84 mm
- net N$8: track 3.26 -> 0.00 mm
- net N$50: track 6.35 -> 9.52 mm
- net N$49: track 6.45 -> 9.63 mm
- net N$55: track 3.68 -> 6.85 mm
- net N$40: track 3.15 -> 0.00 mm
- net N$85: track 4.93 -> 7.80 mm
- net VEXT: track 5.05 -> 7.41 mm
- net N$81: track 3.21 -> 4.89 mm
- net N$59: track 3.21 -> 4.89 mm
- added copper zone on layer 1, net N$11
- added copper zone on layer 1, net N$5
- removed copper zone on layer 1, net N$59
- removed copper zone on layer 1, net N$81
- removed copper zone on layer 1, net VEXT
Other:
- board size 59.7 x 65.4 mm -> 59.7 x 68.6 mm
- board text added: "AIN1+"
- board text added: "AIN1-"
- board text added: "AIN2+"
- board text added: "AIN2-"
- board text added: "DIN1+"
- board text added: "DIN1-"
- board text added: "DIN2+"
- board text added: "DIN2-"
- board text added: "GND"
- board text added: "RESET"
- board text added: "VIN"

Commit message: do
Parts:
- moved SW1 1.00 mm to (7.84, 63.8)
- moved LED1 1.00 mm to (15.3, 61.2)
Connections:
- removed net N$59: CON5.7, R22.1
- removed net N$81: CON5.8, R21.1
- new net N$30: CON5.10, R29.1
- new net N$36: CON5.9, R28.1
- net N$28: now also CON5.8, R22.1; no longer CON5.9, R29.1
- net N$29: now also CON5.7, R21.1; no longer CON5.10, R28.1
Routing:
- net N$36: track 0.00 -> 8.30 mm, vias 0 -> 1
- net N$30: track 0.00 -> 8.12 mm
- net N$81: track 4.89 -> 0.00 mm
- net N$59: track 4.89 -> 0.00 mm
- net N$28: track 4.84 -> 8.18 mm, vias 0 -> 1
- net N$29: track 4.94 -> 8.25 mm
- net N$41: track 58.5 -> 57.4 mm
- net VEXT: track 7.41 -> 8.30 mm
- net N$85: track 7.80 -> 8.40 mm

Commit message: do
Parts:
- added D4, D5: (no value), myparts:SOD123-DIODE
- moved R15 1.66 mm to (28.7, 11.0)
- moved R13 1.65 mm to (22.4, 11.0)
Connections:
- net N$20: now also D4.1
- net N$33: now also D5.1
- net N$49: now also D5.2
- net N$50: now also D4.2
Routing:
- net N$33: track 2.77 -> 5.43 mm
- net N$20: track 2.83 -> 5.43 mm
- net N$85: track 8.40 -> 6.75 mm
- net N$55: track 7.23 -> 5.63 mm
Changed lines of the file:
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@@
 <attribute name="VALUE" x="22.733" y="41.148" size="1.016" layer="27"/>
 </element>
-<element name="R13" library="myparts" package="0805" value="" x="22.352" y="12.7" smashed="yes" rot="R180">
-<attribute name="NAME" x="22.337" y="11.28" size="0.8128" layer="25" rot="R180" align="center"/>
-<attribute name="VALUE" x="24.8285" y="12.7635" size="1.016" layer="27" rot="R180"/>
+<element name="R13" library="myparts" package="0805" value="" x="22.352" y="11.049" smashed="yes" rot="R180">
+<attribute name="NAME" x="19.67" y="11.026" size="0.8128" layer="25" rot="R180" align="center"/>
+<attribute name="VALUE" x="24.8285" y="11.1125" size="1.016" layer="27" rot="R180"/>
 </element>
 <element name="R14" library="myparts" package="0603" value="" x="20.32" y="25.654" smashed="yes">
@@
 <attribute name="VALUE" x="16.891" y="25.4" size="1.016" layer="27"/>
 </element>
-<element name="R15" library="myparts" package="0805" value="" x="28.575" y="12.7" smashed="yes" rot="R180">
-<attribute name="NAME" x="28.56" y="11.28" size="0.8128" layer="25" rot="R180" align="center"/>
-<attribute name="VALUE" x="31.0515" y="12.7635" size="1.016" layer="27" rot="R180"/>
+<element name="R15" library="myparts" package="0805" value="" x="28.702" y="11.049" smashed="yes" rot="R180">
+<attribute name="NAME" x="31.354" y="11.026" size="0.8128" layer="25" rot="R180" align="center"/>
+<attribute name="VALUE" x="31.1785" y="11.1125" size="1.016" layer="27" rot="R180"/>
 </element>
 <element name="R16" library="myparts" package="0603" value="" x="26.67" y="25.654" smashed="yes">
@@
 <attribute name="NAME" x="47.864" y="12.296" size="0.8128" layer="25" rot="R180" align="center"/>
 <attribute name="VALUE" x="49.4665" y="11.1125" size="1.016" layer="27" rot="R180"/>
+</element>
+<element name="D4" library="myparts" package="SOD123-DIODE" value="" x="22.352" y="13.081" smashed="yes">
+<attribute name="NAME" x="19.1675" y="12.9925" size="0.8128" layer="25" align="center"/>
+<attribute name="VALUE" x="22.4695" y="13.6275" size="1.016" layer="27" align="center"/>
+</element>
+<element name="D5" library="myparts" package="SOD123-DIODE" value="" x="28.702" y="13.081" smashed="yes">
+<attribute name="NAME" x="31.9945" y="13.1195" size="0.8128" layer="25" align="center"/>
+<attribute name="VALUE" x="28.8195" y="13.6275" size="1.016" layer="27" align="center"/>
 </element>
 </elements>
@@
 <wire x1="35.44973125" y1="49.1458" x2="42.1672" y2="49.1458" width="0.3048" layer="16"/>
 </signal>
-<signal name="N$20">
-<contactref element="R13" pad="2"/>
-<contactref element="IC3" pad="1"/>
-<wire x1="21.082" y1="15.369" x2="21.082" y2="14.351" width="0.8128" layer="1"/>
-<wire x1="21.082" y1="14.351" x2="21.463" y2="13.97" width="0.8128" layer="1"/>
-<wire x1="21.463" y1="13.97" x2="21.463" y2="12.7" width="0.8128" layer="1"/>
-</signal>
-<signal name="N$33">
-<contactref element="R15" pad="2"/>
-<contactref element="IC4" pad="1"/>
-<wire x1="27.432" y1="15.369" x2="27.432" y2="14.351" width="0.8128" layer="1"/>
-<wire x1="27.432" y1="14.351" x2="27.686" y2="14.097" width="0.8128" layer="1"/>
-<wire x1="27.686" y1="14.097" x2="27.686" y2="12.7" width="0.8128" layer="1"/>
-</signal>
 <signal name="N$50">
+<contactref element="CON5" pad="4"/>
+<wire x1="24.13" y1="8.255" x2="24.13" y2="6.477" width="0.8128" layer="1"/>
+<wire x1="24.13" y1="8.255" x2="24.638" y2="8.763" width="0.8128" layer="1"/>
 <contactref element="IC3" pad="2"/>
-<contactref element="CON5" pad="4"/>
-<wire x1="23.622" y1="15.369" x2="23.622" y2="14.732" width="0.8128" layer="1"/>
-<wire x1="23.622" y1="14.732" x2="24.638" y2="13.716" width="0.8128" layer="1"/>
-<wire x1="24.638" y1="13.716" x2="24.638" y2="8.763" width="0.8128" layer="1"/>
-<wire x1="24.13" y1="8.255" x2="24.13" y2="6.477" width="0.8128" layer="1"/>
-<wire x1="24.638" y1="8.763" x2="24.13" y2="8.255" width="0.8128" layer="1"/>
+<contactref element="D4" pad="2"/>
+<wire x1="24.638" y1="8.763" x2="24.638" y2="12.065" width="0.8128" layer="1"/>
+<wire x1="24.1935" y1="12.5095" x2="24.1935" y2="13.081" width="0.8128" layer="1"/>
+<wire x1="24.638" y1="12.065" x2="24.1935" y2="12.5095" width="0.8128" layer="1"/>
+<wire x1="23.622" y1="15.369" x2="23.622" y2="14.478" width="0.8128" layer="1"/>
+<wire x1="24.1935" y1="13.9065" x2="24.1935" y2="13.081" width="0.8128" layer="1"/>
+<wire x1="23.622" y1="14.478" x2="24.1935" y2="13.9065" width="0.8128" layer="1"/>
 </signal>
 <signal name="N$85">
 <contactref element="R13" pad="1"/>
 <contactref element="CON5" pad="3"/>
-<wire x1="23.241" y1="12.7" x2="23.241" y2="9.398" width="0.8128" layer="1"/>
+<wire x1="23.241" y1="11.049" x2="23.241" y2="9.398" width="0.8128" layer="1"/>
 <wire x1="23.241" y1="9.398" x2="22.733" y2="8.89" width="0.8128" layer="1"/>
 <wire x1="22.733" y1="8.89" x2="21.082" y2="8.89" width="0.8128" layer="1"/>
@@
 <signal name="N$49">
 <contactref element="IC4" pad="2"/>
-<wire x1="29.972" y1="15.369" x2="29.972" y2="14.605" width="0.8128" layer="1"/>
-<wire x1="29.972" y1="14.605" x2="30.861" y2="13.716" width="0.8128" layer="1"/>
 <contactref element="CON5" pad="6"/>
-<wire x1="30.861" y1="13.716" x2="30.861" y2="9.398" width="0.8128" layer="1"/>
 <wire x1="31.75" y1="8.509" x2="31.75" y2="6.477" width="0.8128" layer="1"/>
-<wire x1="31.75" y1="8.509" x2="30.861" y2="9.398" width="0.8128" layer="1"/>
+<wire x1="31.75" y1="8.509" x2="30.988" y2="9.271" width="0.8128" layer="1"/>
+<contactref element="D5" pad="2"/>
+<wire x1="30.988" y1="9.271" x2="30.988" y2="12.065" width="0.8128" layer="1"/>
+<wire x1="30.5435" y1="12.5095" x2="30.5435" y2="13.081" width="0.8128" layer="1"/>
+<wire x1="30.988" y1="12.065" x2="30.5435" y2="12.5095" width="0.8128" layer="1"/>
+<wire x1="29.972" y1="15.369" x2="29.972" y2="14.478" width="0.8128" layer="1"/>
+<wire x1="30.5435" y1="13.9065" x2="30.5435" y2="13.081" width="0.8128" layer="1"/>
+<wire x1="29.972" y1="14.478" x2="30.5435" y2="13.9065" width="0.8128" layer="1"/>
 </signal>
 <signal name="N$55">
 <contactref element="R15" pad="1"/>
 <contactref element="CON5" pad="5"/>
-<wire x1="29.464" y1="12.7" x2="29.464" y2="9.398" width="0.8128" layer="1"/>
-<wire x1="29.464" y1="9.398" x2="28.956" y2="8.89" width="0.8128" layer="1"/>
+<wire x1="29.591" y1="11.049" x2="29.591" y2="9.525" width="0.8128" layer="1"/>
+<wire x1="29.591" y1="9.525" x2="28.956" y2="8.89" width="0.8128" layer="1"/>
 <wire x1="28.956" y1="8.89" x2="28.321" y2="8.89" width="0.8128" layer="1"/>
 <wire x1="28.321" y1="8.89" x2="27.94" y2="8.509" width="0.8128" layer="1"/>
@@
 <wire x1="43.18" y1="7.874" x2="43.18" y2="6.477" width="0.8128" layer="16"/>
 </signal>
+<signal name="N$20">
+<contactref element="IC3" pad="1"/>
+<contactref element="R13" pad="2"/>
+<contactref element="D4" pad="1"/>
+<wire x1="21.463" y1="11.049" x2="21.463" y2="13.081" width="0.8128" layer="1"/>
+<wire x1="21.463" y1="13.081" x2="21.463" y2="13.97" width="0.8128" layer="1"/>
+<wire x1="21.082" y1="14.351" x2="21.082" y2="15.369" width="0.8128" layer="1"/>
+<wire x1="21.463" y1="13.97" x2="21.082" y2="14.351" width="0.8128" layer="1"/>
+<wire x1="20.5105" y1="13.081" x2="21.463" y2="13.081" width="0.8128" layer="1"/>
+</signal>
+<signal name="N$33">
+<contactref element="IC4" pad="1"/>
+<contactref element="R15" pad="2"/>
+<contactref element="D5" pad="1"/>
+<wire x1="27.813" y1="11.049" x2="27.813" y2="13.081" width="0.8128" layer="1"/>
+<wire x1="27.813" y1="13.081" x2="27.813" y2="13.97" width="0.8128" layer="1"/>
+<wire x1="27.432" y1="14.351" x2="27.432" y2="15.369" width="0.8128" layer="1"/>
+<wire x1="27.813" y1="13.97" x2="27.432" y2="14.351" width="0.8128" layer="1"/>
+<wire x1="26.8605" y1="13.081" x2="27.813" y2="13.081" width="0.8128" layer="1"/>
+</signal>
 </signals>

Commit message: s
Parts:
- added C28, C29: (no value), myparts:0603
- moved C21 24.8 mm to (35.6, 47.2), turned to 180 degrees
- moved C20 21.9 mm to (29.1, 44.2)
- moved C22 14.3 mm to (20.3, 24.1)
- moved C23 8.08 mm to (26.7, 24.1)
- moved C25 7.90 mm to (33.1, 19.3)
- moved C19 6.65 mm to (29.1, 45.7), turned to 0 degrees
- moved C26 4.67 mm to (37.5, 16.1)
- moved C24 4.62 mm to (33.1, 17.8)
- moved C27 4.62 mm to (40.9, 17.8)
- moved R4 3.09 mm to (26.2, 44.2)
- moved C16 0.51 mm to (35.6, 45.7)
- moved C5 0.51 mm to (32.0, 45.7)
Connections:
- net GND: now also C24.1, C27.1, C28.1; no longer C26.1
- net N$13: now also C19.2, C20.2
- net N$17: now also C29.1; no longer C27.1
- net N$2: now also C21.2; no longer C19.2
- net N$21: now also C29.2; no longer C27.2
- net N$32: now also C23.2; no longer C21.2
- net N$35: now also C22.2; no longer C20.2
- net N$42: now also C27.2, C28.2; no longer C25.2, C26.2
- net N$68: now also C26.2; no longer C24.2
- net N$69: now also C26.1; no longer C24.1
- net N$77: now also C24.2, C25.2; no longer C22.2, C23.2
Routing:
- net GND: track 76.6 -> 80.6 mm
- net N$1: track 8.80 -> 12.3 mm, vias 0 -> 2
- net N$13: track 22.4 -> 25.5 mm
- net N$26: track 26.5 -> 24.7 mm
- net VCC: track 162.7 -> 163.6 mm
- net N$19: track 28.8 -> 28.2 mm
- net N$18: track 26.7 -> 26.1 mm
- net N$31: track 2.93 -> 3.44 mm

Commit message: s
Parts:
- removed D3: (no value), myparts:SOD123-DIODE
- added C30, C31: (no value), myparts:0603
- L1: device myparts:INDUCTOR-0520-0630 -> myparts:INDUCTOR-CDRH127R
- moved C13 5.50 mm to (11.0, 39.2)
- moved C14 5.50 mm to (11.0, 41.1)
- moved F1 5.50 mm to (11.0, 47.8)
- moved C12 5.50 mm to (11.0, 36.8)
- moved C8 5.50 mm to (11.2, 49.7)
- moved D1 5.50 mm to (11.0, 45.3)
- moved L1 3.10 mm to (11.0, 28.2), turned to 0 degrees
- moved C9 2.51 mm to (9.91, 13.3)
- moved D2 2.43 mm to (9.91, 11.0)
- moved C10 1.78 mm to (13.8, 19.4)
- moved IC2 1.78 mm to (11.0, 18.7)
- moved R6 1.78 mm to (13.8, 16.5)
- moved C11 1.78 mm to (8.26, 19.4)
- moved R5 1.78 mm to (15.4, 19.4)
- moved C16 0.64 mm to (34.9, 45.7)
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Connections:
- net GND: now also C30.1, C31.1, CON5.1; no longer CON5.2, D3.2
- net N$57: now also C30.2
- net VCC: now also C31.2; no longer D3.1
- net VEXT: now also CON5.2; no longer CON5.1
Routing:
- net N$56: track 32.1 -> 15.6 mm
- net VCC: track 163.6 -> 154.6 mm
- net N$57: track 34.1 -> 39.9 mm
- net UVCC: track 41.4 -> 35.7 mm, vias 5 -> 3
- net VEXT: track 8.30 -> 11.3 mm
- net N$16: track 24.0 -> 23.1 mm
- net N$41: track 57.5 -> 56.6 mm
- net N$25: track 44.7 -> 44.0 mm
- net N$24: track 45.9 -> 45.2 mm
- net N$14: track 23.7 -> 23.1 mm
- net N$7: track 16.8 -> 17.5 mm
- net N$6: track 12.3 -> 12.9 mm
- net N$2: track 14.5 -> 13.9 mm
- net N$13: track 25.5 -> 24.8 mm
Other:
- board text added: "DC IN"
- board text removed: "VIN"

Commit message: s
Parts:
- removed D5: (no value), myparts:SOD123-DIODE
- added D3: (no value), myparts:SOD123-DIODE
- C12: device myparts:1206 -> myparts:0603
- C14: device myparts:0603 -> myparts:1206
- C15: device myparts:CAPACITOR-SMD-8 -> myparts:0603
- C17: device myparts:0603 -> myparts:CAPACITOR-SMD-8
- moved C31 43.3 mm to (45.2, 16.1)
- moved C30 31.3 mm to (40.9, 19.3)
- moved C23 24.5 mm to (34.9, 47.2), turned to 180 degrees
- moved C16 24.1 mm to (11.0, 42.7)
- moved C22 21.9 mm to (29.1, 44.2)
- moved C12 17.6 mm to (8.26, 19.4), turned to 270 degrees
- moved C24 14.3 mm to (20.3, 24.1)
- moved C17 11.2 mm to (19.8, 42.5)
- moved C15 8.87 mm to (11.0, 41.1)
- moved C25 8.49 mm to (26.2, 24.1)
- moved C27 7.90 mm to (33.1, 19.3)
- moved D4 6.35 mm to (28.7, 13.1)
- moved C18 6.04 mm to (34.9, 45.7)
- moved C21 6.04 mm to (29.1, 45.7), turned to 0 degrees
- moved C10 5.75 mm to (9.91, 15.2), turned to 0 degrees
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Connections:
- removed net N$7: MOD1.2, R10.1, R9.2
- new net N$37: MOD1.4, R10.1, R9.2
- net GND: now also C10.1, C26.1, C29.1; no longer C12.1, C28.1, C31.1
- net N$13: now also C21.2, C22.2; no longer C17.2, C18.2
- net N$17: now also C31.1; no longer C29.1
- net N$2: now also C23.2; no longer C21.2
- net N$20: now also D3.1; no longer D4.1
- net N$21: now also C31.2; no longer C29.2
- net N$32: now also C25.2; no longer C23.2
- net N$33: now also D4.1; no longer D5.1
- net N$35: now also C24.2; no longer C22.2
- net N$42: now also C29.2, C30.2; no longer C27.2, C28.2
- net N$49: now also D4.2; no longer D5.2
- net N$50: now also D3.2; no longer D4.2
- net N$57: now also C10.2; no longer C30.2
- net N$6: now also MOD1.5; no longer MOD1.1
- net N$65: now also C12.2; no longer C11.2
- net N$66: now also C12.1; no longer C11.1
- net N$68: now also C28.2; no longer C26.2
- net N$69: now also C28.1; no longer C26.1
- net N$72: now also C11.1; no longer C10.1
- net N$77: now also C26.2, C27.2; no longer C24.2, C25.2
- net VCC: now also C11.2, C17.2, C18.2; no longer C10.2, C12.2, C31.2
Routing:
- net N$37: track 0.00 -> 19.1 mm
- net N$7: track 17.5 -> 0.00 mm
- net N$56: track 15.6 -> 25.6 mm
- net VCC: track 154.6 -> 162.6 mm, vias 17 -> 18
- net N$6: track 12.9 -> 19.6 mm, vias 0 -> 2
- net N$57: track 39.9 -> 42.5 mm
- net N$26: track 24.8 -> 25.9 mm
- net N$41: track 56.6 -> 57.7 mm
- net VEXT: track 11.3 -> 12.1 mm
- net N$32: track 45.0 -> 45.7 mm
- net UVCC: track 35.7 -> 36.4 mm

Commit message: s
Routing:
- net N$57: vias 2 -> 4
Changed lines of the file:
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@@
 <wire x1="15.24" y1="43.434" x2="15.24" y2="42.418" width="1.27" layer="16"/>
 <wire x1="14.097" y1="44.577" x2="15.24" y2="43.434" width="1.27" layer="16"/>
-<wire x1="15.24" y1="42.418" x2="15.24" y2="37.592" width="1.27" layer="1"/>
 <wire x1="15.367" y1="11.049" x2="11.7475" y2="11.049" width="1.27" layer="1"/>
-<wire x1="15.24" y1="37.592" x2="17.272" y2="35.56" width="1.27" layer="1"/>
-<wire x1="17.272" y1="35.56" x2="17.272" y2="31.242" width="1.27" layer="1"/>
-<wire x1="17.272" y1="31.242" x2="18.034" y2="30.48" width="1.27" layer="1"/>
-<wire x1="18.034" y1="30.48" x2="18.034" y2="13.716" width="1.27" layer="1"/>
-<wire x1="18.034" y1="13.716" x2="15.367" y2="11.049" width="1.27" layer="1"/>
+<wire x1="15.367" y1="11.049" x2="18.034" y2="13.716" width="1.27" layer="1"/>
+<via x="18.034" y="30.607" extent="1-16" drill="0.7"/>
+<wire x1="18.034" y1="13.716" x2="18.034" y2="30.607" width="1.27" layer="1"/>
+<via x="16.383" y="36.195" extent="1-16" drill="0.7"/>
+<wire x1="15.24" y1="37.338" x2="16.383" y2="36.195" width="1.27" layer="1"/>
+<wire x1="15.24" y1="42.418" x2="15.24" y2="37.338" width="1.27" layer="1"/>
+<wire x1="18.034" y1="30.607" x2="16.891" y2="31.75" width="1.27" layer="16"/>
+<wire x1="16.891" y1="35.687" x2="16.383" y2="36.195" width="1.27" layer="16"/>
+<wire x1="16.891" y1="31.75" x2="16.891" y2="35.687" width="1.27" layer="16"/>
 </signal>
 <signal name="N$41">
