File: eagle/daq.sch (EAGLE design)
At the start: 109 parts

Commit message: do
Parts:
- removed BAT1: (no value), myparts:BAT-1220-BC501SM
- removed C19, C20, C21, C30, C31, C8: (no value), myparts:CAPACITOR-0603
- removed CON6: (no value), myparts:KF2EDGR-3.5-6P
- removed F2, F3: (no value), myparts:FUSE-1206
- removed IC10, IC9: (no value), myparts:NUD3105-12-24-60
- removed IC3: (no value), myparts:DS3231M
- removed IC8: (no value), myparts:IC-485-HALF
- removed R15, R18, R35, R36, R37, R38, R39, R4, R40, R43: (no value), myparts:RESISTOR-0603
- removed R41, R42: (no value), myparts:RESISTOR-0805
- removed SW2: (no value), myparts:B3F-3150-52-55
- removed SW3, SW4: (no value), myparts:HFD2-L2
- CON5: device myparts:KF2EDGR-3.5-12P -> myparts:15EDGRC-3.81-10P
- SW1: device myparts:B3F-3150-52-55 -> myparts:BUTTON-4P-SMD-5X5
Connections:
- removed net N$24: IC1.ADC7/PF7, IC9.G_1
- removed net N$26: IC9.D_1, SW3.L1-
- removed net N$28: IC9.D_2, SW3.L2-
- removed net N$29: C8.1, IC1.PE6/AIN0/INT6, R4.1, SW2.1
- removed net N$38: IC1.ADC6/PF6, IC9.G_2
- removed net N$39: CON6.1, SW4.NO1, SW4.NO2
- removed net N$46: CON5.2, F3.1
- removed net N$47: IC8.R, R35.2, R36.2
- removed net N$48: IC8.D, R39.2
- removed net N$51: IC8.B, R40.2, R41.2
- removed net N$52: IC8.A, R42.2, R43.2
- removed net N$53: IC8.!RE, IC8.DE, R37.2, R38.2
- removed net N$54: F3.2, R42.1
- removed net N$58: BAT1.+, C21.2, IC3.VBAT
- removed net N$60: CON5.1, F2.1
- removed net N$61: IC1.PD2/RXD1/INT2, R36.1
- removed net N$62: IC1.PD3/TXD1/INT3, R39.1
- removed net N$63: IC1.ADC8/PD4, R38.1
- removed net N$64: IC10.D_1, SW4.L1-
- removed net N$67: CON6.2, SW4.NC1, SW4.NC2
- removed net N$70: IC3.!INT, R15.1, R18.2
- removed net N$74: CON6.3, SW4.C1, SW4.C2
- removed net N$80: F2.2, R41.1
- removed net N$82: IC10.D_2, SW4.L2-
- removed net N$86: CON6.4, SW3.NO1, SW3.NO2
- removed net N$87: CON6.5, SW3.NC1, SW3.NC2
- removed net N$88: CON6.6, SW3.C1, SW3.C2
- removed net N$90: IC1.ADC5/PF5, IC10.G_1
- removed net N$91: IC1.ADC4/PF4, IC10.G_2
- new net N$36: IC1.PB7/PCINT7, R6.1
- net GND: now also CON5.2; no longer BAT1.-, C19.1, C20.1, C21.1, C30.1, C31.1, C8.2, CON5.11, IC10.S_1, IC10.S_2, IC3.GND, IC8.GND, IC9.S_1, IC9.S_2, R37.1, R40.1, R6.1, SW1.4, SW2.2, SW2.3, SW2.4
- net N$1: now also IC1.ADC1/PF1; no longer IC1.ADC0/PF0
- net N$30: now also CON5.9; no longer CON5.4
- net N$32: now also IC1.PD3/TXD1/INT3; no longer IC1.PCINT5/ADC12/PB5
- net N$35: now also IC1.PD2/RXD1/INT2; no longer IC1.PCINT4/ADC11/PB4
- net N$40: now also CON5.10; no longer CON5.3
- net N$41: now also SW1.4
- net N$45: no longer R15.2
- net N$49: now also CON5.6; no longer CON5.7
- net N$50: now also CON5.4; no longer CON5.9
- net N$55: now also CON5.5; no longer CON5.8
- net N$59: now also CON5.7; no longer CON5.6
- net N$73: no longer IC3.SCL
- net N$79: no longer IC3.SDA
- net N$81: now also CON5.8; no longer CON5.5
- net N$85: now also CON5.3; no longer CON5.10
- net VCC: no longer C19.2, C20.2, C30.2, C31.2, IC3.VCC, IC8.VCC, R18.1, R35.1, R4.2, R43.1, SW3.L1+, SW3.L2+, SW4.L1+, SW4.L2+
- net VEXT: now also CON5.1; no longer CON5.12
Other:
- note removed: "A"
- note removed: "B"
- note removed: "OUT1_C"
- note removed: "OUT1_NC"
- note removed: "OUT1_NO"
- note removed: "OUT2_C"
- note removed: "OUT2_NC"
- note removed: "OUT2_NO"
- moved on the sheet: C16, C17, C18, CON2, CON3, MOD1, R10, R11, R12, R13, R14, R9

Commit message: do
Parts:
- SW1: device myparts:BUTTON-4P-SMD-5X5 -> myparts:B3F-3150-52-55
Connections:
- net GND: now also SW1.4
- net N$41: no longer SW1.4
Changed lines of the file:
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@@
 <part name="GND35" library="myparts" deviceset="GND" device=""/>
 <part name="CON5" library="myparts" deviceset="15EDGRC-3.81-10P" device=""/>
-<part name="SW1" library="myparts" deviceset="BUTTON-4P-SMD-5X5" device=""/>
+<part name="SW1" library="myparts" deviceset="B3F-3150-52-55" device=""/>
 <part name="GND13" library="myparts" deviceset="GND" device=""/>
 <part name="GND24" library="myparts" deviceset="GND" device=""/>
+<part name="GND25" library="myparts" deviceset="GND" device=""/>
 </parts>
 <sheets>
@@
 <attribute name="VALUE" x="-10.414" y="-162.56" size="1.778" layer="96" rot="MR270" align="center-left"/>
 </instance>
-<instance part="SW1" gate="G$1" x="-45.72" y="-53.34" smashed="yes">
-<attribute name="NAME" x="-42.926" y="-49.784" size="1.778" layer="95" align="center-left"/>
-<attribute name="VALUE" x="-42.926" y="-48.006" size="1.778" layer="96" align="center-left"/>
-</instance>
-<instance part="GND13" gate="1" x="-45.72" y="-58.42" smashed="yes">
-<attribute name="VALUE" x="-48.26" y="-61.468" size="1.778" layer="96"/>
-</instance>
-<instance part="GND24" gate="1" x="-33.02" y="-58.42" smashed="yes">
-<attribute name="VALUE" x="-35.56" y="-61.468" size="1.778" layer="96"/>
+<instance part="SW1" gate="G$1" x="40.64" y="71.12" smashed="yes" rot="R180">
+<attribute name="NAME" x="37.846" y="67.564" size="1.778" layer="95" rot="R180" align="center-left"/>
+<attribute name="VALUE" x="37.846" y="65.786" size="1.778" layer="96" rot="R180" align="center-left"/>
+</instance>
+<instance part="GND13" gate="1" x="43.18" y="71.12" smashed="yes" rot="R90">
+<attribute name="VALUE" x="46.228" y="68.58" size="1.778" layer="96" rot="R90"/>
+</instance>
+<instance part="GND24" gate="1" x="25.4" y="73.66" smashed="yes" rot="R270">
+<attribute name="VALUE" x="22.352" y="76.2" size="1.778" layer="96" rot="R270"/>
+</instance>
+<instance part="GND25" gate="1" x="25.4" y="71.12" smashed="yes" rot="R270">
+<attribute name="VALUE" x="22.352" y="73.66" size="1.778" layer="96" rot="R270"/>
 </instance>
 </instances>
@@
 </segment>
 <segment>
+<pinref part="SW1" gate="G$1" pin="3"/>
+<pinref part="GND13" gate="1" pin="GND"/>
+</segment>
+<segment>
 <pinref part="SW1" gate="G$1" pin="2"/>
-<pinref part="GND13" gate="1" pin="GND"/>
-</segment>
-<segment>
-<pinref part="SW1" gate="G$1" pin="3"/>
 <pinref part="GND24" gate="1" pin="GND"/>
+</segment>
+<segment>
+<pinref part="SW1" gate="G$1" pin="4"/>
+<pinref part="GND25" gate="1" pin="GND"/>
 </segment>
 </net>
@@
 <junction x="-20.32" y="-48.26"/>
 <wire x1="-25.4" y1="-40.64" x2="-25.4" y2="-48.26" width="0.1524" layer="91"/>
+<wire x1="-25.4" y1="-48.26" x2="-45.72" y2="-48.26" width="0.1524" layer="91"/>
+<wire x1="-45.72" y1="-48.26" x2="-45.72" y2="-71.12" width="0.1524" layer="91"/>
+<wire x1="-45.72" y1="-71.12" x2="45.72" y2="-71.12" width="0.1524" layer="91"/>
+<wire x1="45.72" y1="-71.12" x2="45.72" y2="73.66" width="0.1524" layer="91"/>
 <pinref part="SW1" gate="G$1" pin="1"/>
-<wire x1="-25.4" y1="-48.26" x2="-33.02" y2="-48.26" width="0.1524" layer="91"/>
-<wire x1="-33.02" y1="-48.26" x2="-45.72" y2="-48.26" width="0.1524" layer="91"/>
-<wire x1="-45.72" y1="-48.26" x2="-45.72" y2="-53.34" width="0.1524" layer="91"/>
-<pinref part="SW1" gate="G$1" pin="4"/>
-<wire x1="-33.02" y1="-53.34" x2="-33.02" y2="-48.26" width="0.1524" layer="91"/>
-<junction x="-33.02" y="-48.26"/>
-</segment>
-</net>
+<wire x1="45.72" y1="73.66" x2="40.64" y2="73.66" width="0.1524" layer="91"/>
+</segment>
+</net>

Commit message: do
Parts:
- removed LED1: (no value), myparts:LED-HOLDER-2P
- removed R6: (no value), myparts:RESISTOR-0603
Connections:
- removed net N$15: LED1.K2, R5.2
- removed net N$30: CON5.9, R31.1, R32.1
- removed net N$36: IC1.PB7/PCINT7, R6.1
- net N$40: now also R31.1, R32.1; no longer R32.2, R33.1
- net N$59: now also R27.1, R28.2; no longer R26.2, R27.2
- net N$8: now also CON5.9, R32.2, R33.1; no longer LED1.K1, R6.2
- net N$81: now also R26.2, R27.2; no longer R27.1, R28.2
- net VCC: no longer LED1.A1, LED1.A2
Other:
- moved on the sheet: R5
Changed lines of the file:
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@@
 <part name="GND26" library="myparts" deviceset="GND" device=""/>
 <part name="SUP2" library="myparts" deviceset="VCC" device=""/>
-<part name="LED1" library="myparts" deviceset="LED-HOLDER-2P" device=""/>
-<part name="R6" library="myparts" deviceset="RESISTOR-0603" device=""/>
-<part name="SUP4" library="myparts" deviceset="VCC" device=""/>
 <part name="R5" library="myparts" deviceset="RESISTOR-0603" device=""/>
 <part name="SUP7" library="myparts" deviceset="VCC" device=""/>
@@
 <attribute name="VALUE" x="-222.885" y="-104.775" size="1.778" layer="96"/>
 </instance>
-<instance part="LED1" gate="G$1" x="-58.42" y="73.66" smashed="yes">
-<attribute name="NAME" x="-54.864" y="76.454" size="1.778" layer="95" align="center-left"/>
-<attribute name="VALUE" x="-56.896" y="77.47" size="1.778" layer="96" align="center-left"/>
-</instance>
-<instance part="R6" gate="G$1" x="-71.12" y="73.66" smashed="yes">
-<attribute name="NAME" x="-66.802" y="76.2" size="1.778" layer="95" align="center-left"/>
-<attribute name="VALUE" x="-68.072" y="77.47" size="1.778" layer="96" align="center-left"/>
-</instance>
-<instance part="SUP4" gate="G$1" x="-43.18" y="73.66" smashed="yes" rot="R270">
-<attribute name="VALUE" x="-41.275" y="75.565" size="1.778" layer="96" rot="R270"/>
-</instance>
-<instance part="R5" gate="G$1" x="-71.12" y="71.12" smashed="yes">
-<attribute name="NAME" x="-66.802" y="68.834" size="1.778" layer="95" align="center-left"/>
-<attribute name="VALUE" x="-68.072" y="74.93" size="1.778" layer="96" align="center-left"/>
-</instance>
-<instance part="SUP7" gate="G$1" x="-43.18" y="71.12" smashed="yes" rot="R270">
-<attribute name="VALUE" x="-41.275" y="73.025" size="1.778" layer="96" rot="R270"/>
+<instance part="R5" gate="G$1" x="-2.54" y="48.26" smashed="yes" rot="R90">
+<attribute name="NAME" x="-0.254" y="52.578" size="1.778" layer="95" rot="R90" align="center-left"/>
+<attribute name="VALUE" x="-6.35" y="51.308" size="1.778" layer="96" rot="R90" align="center-left"/>
+</instance>
+<instance part="SUP7" gate="G$1" x="-2.54" y="76.2" smashed="yes">
+<attribute name="VALUE" x="-4.445" y="78.105" size="1.778" layer="96"/>
 </instance>
 <instance part="IC4" gate="G$1" x="-190.5" y="-104.14" smashed="yes">
@@
 <wire x1="-215.9" y1="-109.22" x2="-210.82" y2="-109.22" width="0.1524" layer="91"/>
 <junction x="-215.9" y="-109.22"/>
-</segment>
-<segment>
-<pinref part="LED1" gate="G$1" pin="A1"/>
-<pinref part="SUP4" gate="G$1" pin="VCC"/>
-</segment>
-<segment>
-<pinref part="LED1" gate="G$1" pin="A2"/>
-<pinref part="SUP7" gate="G$1" pin="VCC"/>
 </segment>
 <segment>
@@
 </segment>
 </net>
-<net name="N$8" class="0">
-<segment>
-<pinref part="LED1" gate="G$1" pin="K1"/>
-<pinref part="R6" gate="G$1" pin="2"/>
-</segment>
-</net>
-<net name="N$15" class="0">
-<segment>
-<pinref part="LED1" gate="G$1" pin="K2"/>
-<pinref part="R5" gate="G$1" pin="2"/>
-</segment>
-</net>
 <net name="N$18" class="0">
 <segment>
@@
 <net name="N$1" class="0">
 <segment>
+<pinref part="IC1" gate="G$1" pin="ADC1/PF1"/>
+<wire x1="-2.54" y1="48.26" x2="-2.54" y2="35.56" width="0.1524" layer="91"/>
 <pinref part="R5" gate="G$1" pin="1"/>
-<wire x1="-71.12" y1="63.5" x2="-71.12" y2="71.12" width="0.1524" layer="91"/>
-<wire x1="-71.12" y1="63.5" x2="-2.54" y2="63.5" width="0.1524" layer="91"/>
-<pinref part="IC1" gate="G$1" pin="ADC1/PF1"/>
-<wire x1="-2.54" y1="63.5" x2="-2.54" y2="35.56" width="0.1524" layer="91"/>
 </segment>
 </net>
@@
 <wire x1="-7.62" y1="-104.14" x2="-15.24" y2="-104.14" width="0.1524" layer="91"/>
 <pinref part="IC7" gate="G$1" pin="IN+"/>
-</segment>
-</net>
-<net name="N$30" class="0">
-<segment>
-<pinref part="R31" gate="G$1" pin="1"/>
-<pinref part="R32" gate="G$1" pin="1"/>
-<wire x1="10.16" y1="-99.06" x2="15.24" y2="-99.06" width="0.1524" layer="91"/>
-<junction x="10.16" y="-99.06"/>
-<pinref part="CON5" gate="G$1" pin="9"/>
-<wire x1="15.24" y1="-99.06" x2="15.24" y2="-157.48" width="0.1524" layer="91"/>
 </segment>
 </net>
@@
 <net name="N$40" class="0">
 <segment>
-<pinref part="R33" gate="G$1" pin="1"/>
-<pinref part="R32" gate="G$1" pin="2"/>
-<wire x1="10.16" y1="-111.76" x2="17.78" y2="-111.76" width="0.1524" layer="91"/>
-<junction x="10.16" y="-111.76"/>
 <pinref part="CON5" gate="G$1" pin="10"/>
-<wire x1="17.78" y1="-111.76" x2="17.78" y2="-157.48" width="0.1524" layer="91"/>
+<wire x1="17.78" y1="-99.06" x2="17.78" y2="-157.48" width="0.1524" layer="91"/>
+<pinref part="R31" gate="G$1" pin="1"/>
+<pinref part="R32" gate="G$1" pin="1"/>
+<wire x1="17.78" y1="-99.06" x2="10.16" y2="-99.06" width="0.1524" layer="91"/>
+<junction x="10.16" y="-99.06"/>
 </segment>
 </net>
 <net name="N$59" class="0">
 <segment>
-<pinref part="R27" gate="G$1" pin="2"/>
-<pinref part="R26" gate="G$1" pin="2"/>
-<wire x1="-66.04" y1="-99.06" x2="-60.96" y2="-99.06" width="0.1524" layer="91"/>
-<junction x="-66.04" y="-99.06"/>
-<wire x1="-60.96" y1="-99.06" x2="-60.96" y2="-139.7" width="0.1524" layer="91"/>
 <wire x1="-60.96" y1="-139.7" x2="10.16" y2="-139.7" width="0.1524" layer="91"/>
 <pinref part="CON5" gate="G$1" pin="7"/>
 <wire x1="10.16" y1="-139.7" x2="10.16" y2="-157.48" width="0.1524" layer="91"/>
+<pinref part="R27" gate="G$1" pin="1"/>
+<pinref part="R28" gate="G$1" pin="2"/>
+<wire x1="-60.96" y1="-139.7" x2="-60.96" y2="-111.76" width="0.1524" layer="91"/>
+<wire x1="-60.96" y1="-111.76" x2="-66.04" y2="-111.76" width="0.1524" layer="91"/>
+<junction x="-66.04" y="-111.76"/>
 </segment>
 </net>
@@
 <net name="N$81" class="0">
 <segment>
-<pinref part="R27" gate="G$1" pin="1"/>
-<pinref part="R28" gate="G$1" pin="2"/>
-<junction x="-66.04" y="-111.76"/>
-<wire x1="-66.04" y1="-111.76" x2="-58.42" y2="-111.76" width="0.1524" layer="91"/>
 <wire x1="-58.42" y1="-137.16" x2="12.7" y2="-137.16" width="0.1524" layer="91"/>
-<wire x1="-58.42" y1="-111.76" x2="-58.42" y2="-137.16" width="0.1524" layer="91"/>
+<wire x1="-58.42" y1="-99.06" x2="-58.42" y2="-137.16" width="0.1524" layer="91"/>
 <pinref part="CON5" gate="G$1" pin="8"/>
 <wire x1="12.7" y1="-137.16" x2="12.7" y2="-157.48" width="0.1524" layer="91"/>
-</segment>
-</net>
-<net name="N$36" class="0">
-<segment>
-<pinref part="R6" gate="G$1" pin="1"/>
-<wire x1="-71.12" y1="73.66" x2="-78.74" y2="73.66" width="0.1524" layer="91"/>
-<pinref part="IC1" gate="G$1" pin="PB7/PCINT7"/>
-<wire x1="-12.7" y1="-35.56" x2="-12.7" y2="-38.1" width="0.1524" layer="91"/>
-<wire x1="-12.7" y1="-38.1" x2="-78.74" y2="-38.1" width="0.1524" layer="91"/>
-<wire x1="-78.74" y1="-38.1" x2="-78.74" y2="73.66" width="0.1524" layer="91"/>
-</segment>
-</net>
+<pinref part="R27" gate="G$1" pin="2"/>
+<pinref part="R26" gate="G$1" pin="2"/>
+<wire x1="-58.42" y1="-99.06" x2="-66.04" y2="-99.06" width="0.1524" layer="91"/>
+<junction x="-66.04" y="-99.06"/>
+</segment>
+</net>
+<net name="N$8" class="0">
+<segment>
+<pinref part="R33" gate="G$1" pin="1"/>
+<pinref part="R32" gate="G$1" pin="2"/>
+<pinref part="CON5" gate="G$1" pin="9"/>
+<wire x1="10.16" y1="-111.76" x2="15.24" y2="-111.76" width="0.1524" layer="91"/>
+<wire x1="15.24" y1="-111.76" x2="15.24" y2="-157.48" width="0.1524" layer="91"/>
+<junction x="10.16" y="-111.76"/>
+</segment>
+</net>

Commit message: do
Connections:
- new net N$26: R5.2
Changed lines of the file:
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@@
+</segment>
+</net>
+<net name="N$26" class="0">
+<segment>
+<pinref part="R5" gate="G$1" pin="2"/>
+<wire x1="-2.54" y1="60.96" x2="-2.54" y2="63.5" width="0.1524" layer="91"/>
 </segment>
 </net>

Commit message: do
Parts:
- added LED1: (no value), myparts:LED-3MM-RA
Connections:
- net N$26: now also LED1.K
- net VCC: now also LED1.A
Changed lines of the file:
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@@
 <part name="GND24" library="myparts" deviceset="GND" device=""/>
 <part name="GND25" library="myparts" deviceset="GND" device=""/>
+<part name="LED1" library="myparts" deviceset="LED-3MM-RA" device=""/>
 </parts>
 <sheets>
@@
 <attribute name="VALUE" x="22.352" y="73.66" size="1.778" layer="96" rot="R270"/>
 </instance>
+<instance part="LED1" gate="G$1" x="-2.54" y="60.96" smashed="yes" rot="R90">
+<attribute name="NAME" x="-4.572" y="62.484" size="1.778" layer="95" rot="R90" align="center-left"/>
+<attribute name="VALUE" x="-6.35" y="62.484" size="1.778" layer="96" rot="R90" align="center-left"/>
+</instance>
 </instances>
 <busses>
@@
 <pinref part="SUP22" gate="G$1" pin="VCC"/>
 <pinref part="R30" gate="G$1" pin="1"/>
+</segment>
+<segment>
+<pinref part="SUP7" gate="G$1" pin="VCC"/>
+<pinref part="LED1" gate="G$1" pin="A"/>
 </segment>
 </net>
@@
 <segment>
 <pinref part="R5" gate="G$1" pin="2"/>
-<wire x1="-2.54" y1="60.96" x2="-2.54" y2="63.5" width="0.1524" layer="91"/>
-</segment>
-</net>
+<pinref part="LED1" gate="G$1" pin="K"/>
+</segment>
+</net>

Commit message: do
Parts:
- removed C28, C29, C33: (no value), myparts:CAPACITOR-0603
- removed C32: (no value), myparts:CAPACITOR-SMD-8
- removed IC7: (no value), myparts:INA226
- removed R31, R33, R34: (no value), myparts:RESISTOR-0603
- removed R32: (no value), myparts:RESISTOR-1206
- added C19, C20, C21, C8: (no value), myparts:CAPACITOR-0603
- added IC3: (no value), myparts:OPTO-SMD
- added R15: (no value), myparts:RESISTOR-0805
- added R18, R4, R6: (no value), myparts:RESISTOR-0603
- C10, C14: device myparts:CAPACITOR-1206 -> myparts:CAPACITOR-0603
- C12, C9: device myparts:CAPACITOR-0603 -> myparts:CAPACITOR-1206
- C15: device myparts:CAPACITOR-0603 -> myparts:CAPACITOR-SMD-8
- IC5: device myparts:OPTO-SMD -> myparts:INA226
- R13: device myparts:RESISTOR-0603 -> myparts:RESISTOR-0805
- R20, R26: device myparts:RESISTOR-0603 -> myparts:RESISTOR-1206
- R21, R23: device myparts:RESISTOR-0805 -> myparts:RESISTOR-0603
- R27: device myparts:RESISTOR-1206 -> myparts:RESISTOR-0603
Connections:
- net GND: now also C12.1, C19.1, C20.1, C21.1, C26.1, C8.1, IC3.E, IC5.A0, IC5.A1, IC5.GND, R6.1; no longer C10.1, C24.1, C27.1, C28.1, C32.1, C33.1, IC5.E, IC6.A0, IC7.A1, IC7.GND, R8.1
- net N$1: now also R4.1; no longer R5.1
- net N$13: now also C18.2, R8.2; no longer C16.2, R14.2
- net N$14: now also R7.1; no longer R9.1
- net N$16: now also R9.1; no longer R11.1
- net N$17: now also C27.1, IC6.IN-, IC6.VBUS, R27.2; no longer C29.1, IC7.IN-, IC7.VBUS, R33.2
- net N$2: now also C19.2, R11.1, R12.1; no longer C18.2, R13.1, R14.1
- net N$20: now also IC3.A, R13.2; no longer IC4.A, R21.2
- net N$21: now also C27.2, IC6.IN+, R25.2; no longer C29.2, IC7.IN+, R31.2
- net N$22: now also R11.2; no longer R13.2
- net N$23: now also IC5.ALR, R17.1, R18.2; no longer IC6.ALR, R16.1, R25.2
- net N$25: now also IC6.ALR, R23.1, R24.2; no longer IC7.ALR, R17.1, R30.2
- net N$26: now also R4.2; no longer R5.2
- net N$27: now also R28.2; no longer R34.2
- net N$3: now also R23.2; no longer R17.2
- net N$32: now also C21.2, IC4.C, R16.2; no longer C23.2, IC5.C, R24.2
- net N$33: now also IC4.A, R15.2; no longer IC5.A, R23.2
- net N$35: now also C20.2, IC3.C, R14.2; no longer C22.2, IC4.C, R22.2
- net N$40: now also R25.1, R26.1; no longer R31.1, R32.1
- net N$42: now also C25.2, C26.2, IC6.VS; no longer C27.2, C28.2, IC7.VS
- net N$49: now also IC4.K; no longer IC5.K
- net N$50: now also IC3.K; no longer IC4.K
- net N$55: now also R15.1; no longer R23.1
- net N$57: now also C9.2; no longer C10.2
- net N$59: now also R20.1, R21.2; no longer R27.1, R28.2
- net N$6: now also R7.2, R8.1; no longer R10.1, R9.2
- net N$65: now also C11.2; no longer C12.2
- net N$66: now also C11.1; no longer C12.1
- net N$68: now also C24.2, IC5.IN+, R19.1; no longer C26.2, IC6.IN+, R26.1
- net N$69: now also C24.1, IC5.IN-, IC5.VBUS, R21.1; no longer C26.1, IC6.IN-, IC6.VBUS, R28.1
- net N$7: now also R10.1, R9.2; no longer R11.2, R12.1
- net N$71: now also R22.2; no longer R29.2
- net N$72: now also C10.1, R5.2, R6.2; no longer C11.1, R7.2, R8.2
- net N$73: now also IC5.SCL, R30.2; no longer IC7.SCL, R20.2
- net N$77: now also C22.2, C23.2, IC5.VS; no longer C24.2, C25.2, IC6.VS
- net N$79: now also IC5.SDA, R29.2; no longer IC7.SDA, R19.2
- net N$8: now also R26.2, R27.1; no longer R32.2, R33.1
- net N$81: now also R19.2, R20.2; no longer R26.2, R27.2
- net N$85: now also R13.1; no longer R21.1
- net N$9: now also R17.2; no longer R16.2
- net UVCC: now also C8.2; no longer C9.2
- net VCC: now also C10.2, C12.2, C16.2, IC6.A0, R14.1, R16.1, R18.1, R28.1, R5.1; no longer C11.2, C32.2, C33.2, IC7.A0, R19.1, R20.1, R25.1, R34.1, R7.1
Other:
- note added: "RESET"
- moved on the sheet: C10, C11, C12, C13, C14, C16, C17, C18, C22, C23, C24, C25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

Commit message: do
Parts:
- removed R29, R30: (no value), myparts:RESISTOR-0603
- R19, R24: device myparts:RESISTOR-0603 -> myparts:RESISTOR-1206
- R20, R26: device myparts:RESISTOR-1206 -> myparts:RESISTOR-0603
Connections:
- removed net N$25: IC6.ALR, R23.1, R24.2
- new net N$15: IC1.PCINT5/ADC12/PB5, IC6.ALR, R22.2
- net N$17: now also R25.2; no longer R27.2
- net N$21: now also R23.2; no longer R25.2
- net N$23: now also IC1.PCINT4/ADC11/PB4, R17.2; no longer R17.1, R18.2
- net N$27: now also R26.2; no longer R28.2
- net N$3: no longer R23.2
- net N$40: now also R23.1, R24.1; no longer R25.1, R26.1
- net N$59: now also R19.1, R20.2; no longer R20.1, R21.2
- net N$68: now also R18.1; no longer R19.1
- net N$69: now also R20.1; no longer R21.1
- net N$71: now also R21.2; no longer R22.2
- net N$73: now also R28.2; no longer R30.2
- net N$79: now also R27.2; no longer R29.2
- net N$8: now also R24.2, R25.1; no longer R26.2, R27.1
- net N$81: now also R18.2; no longer R20.2
- net N$9: no longer R17.2
- net VCC: now also R17.1, R21.1, R26.1, R27.1; no longer R18.1, R24.1, R29.1, R30.1
Other:
- moved on the sheet: R17, R18, R19, R20, R21, R22, R23, R24, R25, R26, R27, R28
