File: eagle/daq.sch (EAGLE design)
At the start: 77 parts

Commit message: do
Connections:
- removed net N$11: CON2.1, IC1.PC6
- removed net N$5: CON2.2, IC1.PC7
- new net N$24: CON2.1, IC1.PD3/TXD1/INT3
- new net N$25: CON2.2, IC1.PD2/RXD1/INT2
- net N$15: now also IC1.ADC10/PD7; no longer IC1.PCINT5/ADC12/PB5
- net N$23: now also IC1.ADC9/PD6; no longer IC1.PCINT4/ADC11/PB4
- net N$32: now also IC1.PCINT5/ADC12/PB5; no longer IC1.PD3/TXD1/INT3
- net N$35: now also IC1.PCINT4/ADC11/PB4; no longer IC1.PD2/RXD1/INT2
Other:
- moved on the sheet: C17, C18, C19, CON2, CON3, MOD1, R10, R11, R12, R7, R8, R9

Commit message: do
Parts:
- added R29: (no value), myparts:RESISTOR-0805
- added R30, R31, R32: (no value), myparts:RESISTOR-0603
- R19: device myparts:RESISTOR-1206 -> myparts:RESISTOR-0805
- R21, R22, R26, R28: device myparts:RESISTOR-0603 -> myparts:RESISTOR-0805
- R24: device myparts:RESISTOR-1206 -> myparts:RESISTOR-0603
Connections:
- new net N$11: R18.2, R19.2, R21.2
- new net N$28: CON5.9, R29.1
- new net N$29: CON5.10, R28.1
- new net N$5: R19.1, R20.2, R22.2
- net N$15: now also R24.2; no longer R22.2
- net N$17: now also R27.2; no longer R25.2
- net N$21: now also R25.2; no longer R23.2
- net N$27: now also R30.2; no longer R26.2
- net N$40: now also R25.1, R26.2, R28.2; no longer CON5.10, R23.1, R24.1
- net N$59: now also R22.1; no longer R19.1, R20.2
- net N$71: now also R23.2; no longer R21.2
- net N$73: now also R32.2; no longer R28.2
- net N$79: now also R31.2; no longer R27.2
- net N$8: now also R26.1, R27.1, R29.2; no longer CON5.9, R24.2, R25.1
- net N$81: now also R21.1; no longer R18.2, R19.2
- net VCC: now also R23.1, R24.1, R30.1, R31.1, R32.1; no longer R21.1, R22.1, R26.1, R27.1, R28.1
Other:
- moved on the sheet: R21, R22, R23, R24, R25, R26, R27, R28

Commit message: do
Connections:
- removed net N$59: CON5.7, R22.1
- removed net N$81: CON5.8, R21.1
- new net N$30: CON5.10, R29.1
- new net N$36: CON5.9, R28.1
- net N$28: now also CON5.8, R22.1; no longer CON5.9, R29.1
- net N$29: now also CON5.7, R21.1; no longer CON5.10, R28.1
Changed lines of the file:
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@@
 <setting verticaltext="up"/>
 </settings>
-<grid distance="0.02" unitdist="inch" unit="inch" style="lines" multiple="1" display="no" altdistance="0.01" altunitdist="inch" altunit="inch"/>
+<grid distance="0.1" unitdist="inch" unit="inch" style="lines" multiple="1" display="no" altdistance="0.01" altunitdist="inch" altunit="inch"/>
 <layers>
 <layer number="1" name="Top" color="4" fill="1" visible="no" active="no"/>
@@
 </segment>
 </net>
-<net name="N$59" class="0">
-<segment>
-<wire x1="-60.96" y1="-139.7" x2="10.16" y2="-139.7" width="0.1524" layer="91"/>
-<pinref part="CON5" gate="G$1" pin="7"/>
-<wire x1="10.16" y1="-139.7" x2="10.16" y2="-157.48" width="0.1524" layer="91"/>
-<pinref part="R22" gate="G$1" pin="1"/>
-<wire x1="-60.96" y1="-129.54" x2="-60.96" y2="-139.7" width="0.1524" layer="91"/>
-</segment>
-</net>
 <net name="N$68" class="0">
 <segment>
@@
 </segment>
 </net>
-<net name="N$81" class="0">
-<segment>
-<wire x1="-58.42" y1="-137.16" x2="12.7" y2="-137.16" width="0.1524" layer="91"/>
-<pinref part="CON5" gate="G$1" pin="8"/>
-<wire x1="12.7" y1="-137.16" x2="12.7" y2="-157.48" width="0.1524" layer="91"/>
-<pinref part="R21" gate="G$1" pin="1"/>
-<wire x1="-58.42" y1="-129.54" x2="-58.42" y2="-137.16" width="0.1524" layer="91"/>
-</segment>
-</net>
 <net name="N$8" class="0">
 <segment>
@@
 <net name="N$28" class="0">
 <segment>
+<pinref part="R22" gate="G$1" pin="1"/>
+<wire x1="-60.96" y1="-129.54" x2="-60.96" y2="-139.7" width="0.1524" layer="91"/>
+<wire x1="-60.96" y1="-139.7" x2="12.7" y2="-139.7" width="0.1524" layer="91"/>
+<pinref part="CON5" gate="G$1" pin="8"/>
+<wire x1="12.7" y1="-139.7" x2="12.7" y2="-157.48" width="0.1524" layer="91"/>
+</segment>
+</net>
+<net name="N$29" class="0">
+<segment>
+<pinref part="R21" gate="G$1" pin="1"/>
+<wire x1="-58.42" y1="-129.54" x2="-58.42" y2="-137.16" width="0.1524" layer="91"/>
+<wire x1="-58.42" y1="-137.16" x2="10.16" y2="-137.16" width="0.1524" layer="91"/>
+<pinref part="CON5" gate="G$1" pin="7"/>
+<wire x1="10.16" y1="-137.16" x2="10.16" y2="-157.48" width="0.1524" layer="91"/>
+</segment>
+</net>
+<net name="N$30" class="0">
+<segment>
 <pinref part="R29" gate="G$1" pin="1"/>
+<wire x1="15.24" y1="-129.54" x2="15.24" y2="-134.62" width="0.1524" layer="91"/>
+<wire x1="15.24" y1="-134.62" x2="17.78" y2="-134.62" width="0.1524" layer="91"/>
+<pinref part="CON5" gate="G$1" pin="10"/>
+<wire x1="17.78" y1="-134.62" x2="17.78" y2="-157.48" width="0.1524" layer="91"/>
+</segment>
+</net>
+<net name="N$36" class="0">
+<segment>
+<pinref part="R28" gate="G$1" pin="1"/>
+<wire x1="17.78" y1="-129.54" x2="17.78" y2="-132.08" width="0.1524" layer="91"/>
+<wire x1="17.78" y1="-132.08" x2="12.7" y2="-132.08" width="0.1524" layer="91"/>
+<wire x1="12.7" y1="-132.08" x2="12.7" y2="-137.16" width="0.1524" layer="91"/>
 <pinref part="CON5" gate="G$1" pin="9"/>
-<wire x1="15.24" y1="-129.54" x2="15.24" y2="-157.48" width="0.1524" layer="91"/>
-</segment>
-</net>
-<net name="N$29" class="0">
-<segment>
-<pinref part="R28" gate="G$1" pin="1"/>
-<pinref part="CON5" gate="G$1" pin="10"/>
-<wire x1="17.78" y1="-129.54" x2="17.78" y2="-157.48" width="0.1524" layer="91"/>
-</segment>
-</net>
+<wire x1="12.7" y1="-137.16" x2="15.24" y2="-137.16" width="0.1524" layer="91"/>
+<wire x1="15.24" y1="-137.16" x2="15.24" y2="-157.48" width="0.1524" layer="91"/>
+</segment>
+</net>

Commit message: do
Parts:
- added D4, D5: (no value), myparts:DIODE-SCHOTTKY
Connections:
- net N$20: now also D4.K
- net N$33: now also D5.K
- net N$49: now also D5.A
- net N$50: now also D4.A
Other:
- moved on the sheet: R13, R15
Changed lines of the file:
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@@
 <setting verticaltext="up"/>
 </settings>
-<grid distance="0.1" unitdist="inch" unit="inch" style="lines" multiple="1" display="no" altdistance="0.01" altunitdist="inch" altunit="inch"/>
+<grid distance="0.02" unitdist="inch" unit="inch" style="lines" multiple="1" display="no" altdistance="0.01" altunitdist="inch" altunit="inch"/>
 <layers>
 <layer number="1" name="Top" color="4" fill="1" visible="no" active="no"/>
@@
 <part name="R29" library="myparts" deviceset="RESISTOR-0805" device=""/>
 <part name="R28" library="myparts" deviceset="RESISTOR-0805" device=""/>
+<part name="D4" library="myparts" deviceset="DIODE-SCHOTTKY" device=""/>
+<part name="D5" library="myparts" deviceset="DIODE-SCHOTTKY" device=""/>
 </parts>
 <sheets>
@@
 <attribute name="VALUE" x="-160.02" y="-96.52" size="1.778" layer="94"/>
 </instance>
-<instance part="R13" gate="G$1" x="-203.2" y="-116.84" smashed="yes" rot="R90">
-<attribute name="NAME" x="-205.232" y="-112.776" size="1.778" layer="95" rot="R90" align="center-left"/>
-<attribute name="VALUE" x="-207.01" y="-113.792" size="1.778" layer="96" rot="R90" align="center-left"/>
-</instance>
-<instance part="R15" gate="G$1" x="-167.64" y="-116.84" smashed="yes" rot="R90">
-<attribute name="NAME" x="-169.672" y="-112.776" size="1.778" layer="95" rot="R90" align="center-left"/>
-<attribute name="VALUE" x="-171.45" y="-113.792" size="1.778" layer="96" rot="R90" align="center-left"/>
+<instance part="R13" gate="G$1" x="-203.2" y="-139.7" smashed="yes" rot="R90">
+<attribute name="NAME" x="-205.232" y="-135.636" size="1.778" layer="95" rot="R90" align="center-left"/>
+<attribute name="VALUE" x="-207.01" y="-136.652" size="1.778" layer="96" rot="R90" align="center-left"/>
+</instance>
+<instance part="R15" gate="G$1" x="-167.64" y="-139.7" smashed="yes" rot="R90">
+<attribute name="NAME" x="-169.672" y="-135.636" size="1.778" layer="95" rot="R90" align="center-left"/>
+<attribute name="VALUE" x="-171.45" y="-136.652" size="1.778" layer="96" rot="R90" align="center-left"/>
 </instance>
 <instance part="R14" gate="G$1" x="-175.26" y="-91.44" smashed="yes" rot="R270">
@@
 <attribute name="NAME" x="19.812" y="-125.984" size="1.778" layer="95" rot="R90" align="center-left"/>
 <attribute name="VALUE" x="13.97" y="-126.492" size="1.778" layer="96" rot="R90" align="center-left"/>
+</instance>
+<instance part="D4" gate="G$1" x="-195.58" y="-124.46" smashed="yes" rot="R90">
+<attribute name="NAME" x="-198.12" y="-119.888" size="1.778" layer="95" rot="R90" align="center-left"/>
+<attribute name="VALUE" x="-199.39" y="-122.936" size="1.778" layer="96" rot="R90" align="center-left"/>
+</instance>
+<instance part="D5" gate="G$1" x="-160.02" y="-124.46" smashed="yes" rot="R90">
+<attribute name="NAME" x="-162.56" y="-119.888" size="1.778" layer="95" rot="R90" align="center-left"/>
+<attribute name="VALUE" x="-163.83" y="-122.936" size="1.778" layer="96" rot="R90" align="center-left"/>
 </instance>
 </instances>
@@
 </segment>
 </net>
-<net name="N$20" class="0">
-<segment>
-<pinref part="R13" gate="G$1" pin="2"/>
-<pinref part="IC3" gate="G$1" pin="A"/>
-<wire x1="-203.2" y1="-104.14" x2="-200.66" y2="-104.14" width="0.1524" layer="91"/>
-</segment>
-</net>
-<net name="N$33" class="0">
-<segment>
-<pinref part="R15" gate="G$1" pin="2"/>
-<pinref part="IC4" gate="G$1" pin="A"/>
-<wire x1="-167.64" y1="-104.14" x2="-165.1" y2="-104.14" width="0.1524" layer="91"/>
-</segment>
-</net>
 <net name="N$50" class="0">
 <segment>
-<pinref part="IC3" gate="G$1" pin="K"/>
-<wire x1="-200.66" y1="-106.68" x2="-200.66" y2="-147.32" width="0.1524" layer="91"/>
 <wire x1="-200.66" y1="-147.32" x2="2.54" y2="-147.32" width="0.1524" layer="91"/>
 <pinref part="CON5" gate="G$1" pin="4"/>
 <wire x1="2.54" y1="-147.32" x2="2.54" y2="-157.48" width="0.1524" layer="91"/>
+<pinref part="IC3" gate="G$1" pin="K"/>
+<wire x1="-200.66" y1="-147.32" x2="-200.66" y2="-111.76" width="0.1524" layer="91"/>
+<pinref part="D4" gate="G$1" pin="A"/>
+<wire x1="-200.66" y1="-111.76" x2="-200.66" y2="-106.68" width="0.1524" layer="91"/>
+<wire x1="-195.58" y1="-111.76" x2="-200.66" y2="-111.76" width="0.1524" layer="91"/>
+<junction x="-200.66" y="-111.76"/>
 </segment>
 </net>
@@
 <segment>
 <pinref part="R13" gate="G$1" pin="1"/>
-<wire x1="-203.2" y1="-116.84" x2="-203.2" y2="-149.86" width="0.1524" layer="91"/>
+<wire x1="-203.2" y1="-139.7" x2="-203.2" y2="-149.86" width="0.1524" layer="91"/>
 <wire x1="-203.2" y1="-149.86" x2="0" y2="-149.86" width="0.1524" layer="91"/>
 <pinref part="CON5" gate="G$1" pin="3"/>
@@
 <segment>
 <pinref part="IC4" gate="G$1" pin="K"/>
-<wire x1="-165.1" y1="-106.68" x2="-165.1" y2="-142.24" width="0.1524" layer="91"/>
+<wire x1="-165.1" y1="-106.68" x2="-165.1" y2="-111.76" width="0.1524" layer="91"/>
+<wire x1="-165.1" y1="-111.76" x2="-165.1" y2="-142.24" width="0.1524" layer="91"/>
 <wire x1="-165.1" y1="-142.24" x2="7.62" y2="-142.24" width="0.1524" layer="91"/>
 <pinref part="CON5" gate="G$1" pin="6"/>
 <wire x1="7.62" y1="-142.24" x2="7.62" y2="-157.48" width="0.1524" layer="91"/>
+<pinref part="D5" gate="G$1" pin="A"/>
+<wire x1="-160.02" y1="-111.76" x2="-165.1" y2="-111.76" width="0.1524" layer="91"/>
+<junction x="-165.1" y="-111.76"/>
 </segment>
 </net>
@@
 <segment>
 <pinref part="R15" gate="G$1" pin="1"/>
-<wire x1="-167.64" y1="-116.84" x2="-167.64" y2="-144.78" width="0.1524" layer="91"/>
+<wire x1="-167.64" y1="-139.7" x2="-167.64" y2="-144.78" width="0.1524" layer="91"/>
 <wire x1="-167.64" y1="-144.78" x2="5.08" y2="-144.78" width="0.1524" layer="91"/>
 <pinref part="CON5" gate="G$1" pin="5"/>
@@
 </segment>
 </net>
+<net name="N$20" class="0">
+<segment>
+<pinref part="IC3" gate="G$1" pin="A"/>
+<pinref part="R13" gate="G$1" pin="2"/>
+<wire x1="-200.66" y1="-104.14" x2="-203.2" y2="-104.14" width="0.1524" layer="91"/>
+<wire x1="-203.2" y1="-104.14" x2="-203.2" y2="-124.46" width="0.1524" layer="91"/>
+<pinref part="D4" gate="G$1" pin="K"/>
+<wire x1="-203.2" y1="-124.46" x2="-203.2" y2="-127" width="0.1524" layer="91"/>
+<wire x1="-195.58" y1="-124.46" x2="-203.2" y2="-124.46" width="0.1524" layer="91"/>
+<junction x="-203.2" y="-124.46"/>
+</segment>
+</net>
+<net name="N$33" class="0">
+<segment>
+<pinref part="IC4" gate="G$1" pin="A"/>
+<pinref part="R15" gate="G$1" pin="2"/>
+<wire x1="-165.1" y1="-104.14" x2="-167.64" y2="-104.14" width="0.1524" layer="91"/>
+<wire x1="-167.64" y1="-104.14" x2="-167.64" y2="-124.46" width="0.1524" layer="91"/>
+<pinref part="D5" gate="G$1" pin="K"/>
+<wire x1="-167.64" y1="-124.46" x2="-167.64" y2="-127" width="0.1524" layer="91"/>
+<wire x1="-160.02" y1="-124.46" x2="-167.64" y2="-124.46" width="0.1524" layer="91"/>
+<junction x="-167.64" y="-124.46"/>
+</segment>
+</net>

Commit message: s
Parts:
- added C28, C29: (no value), myparts:CAPACITOR-0603
Connections:
- net GND: now also C24.1, C27.1, C28.1; no longer C26.1
- net N$13: now also C19.2, C20.2
- net N$17: now also C29.1; no longer C27.1
- net N$2: now also C21.2; no longer C19.2
- net N$21: now also C29.2; no longer C27.2
- net N$32: now also C23.2; no longer C21.2
- net N$35: now also C22.2; no longer C20.2
- net N$42: now also C27.2, C28.2; no longer C25.2, C26.2
- net N$68: now also C26.2; no longer C24.2
- net N$69: now also C26.1; no longer C24.1
- net N$77: now also C24.2, C25.2; no longer C22.2, C23.2
Other:
- moved on the sheet: C17, C18, C19, C20, C21, C22, C23, C24, C25, C26, C27

Commit message: s
Parts:
- removed D3: (no value), myparts:ZENER-SOD123
- added C30, C31: (no value), myparts:CAPACITOR-0603
- L1: device myparts:INDUCTOR-0520-0630 -> myparts:INDUCTOR-CDRH127R
Connections:
- net GND: now also C30.1, C31.1, CON5.1; no longer CON5.2, D3.A
- net N$57: now also C30.2
- net VCC: now also C31.2; no longer D3.K
- net VEXT: now also CON5.2; no longer CON5.1
Other:
- note added: "DC IN"
- note removed: "VIN"
- moved on the sheet: C10, C15, C16, C8, D1, D2, F1, R5, R6

Commit message: s
Parts:
- removed D5: (no value), myparts:DIODE-SCHOTTKY
- added D3: (no value), myparts:DIODE-SCHOTTKY
- C12: device myparts:CAPACITOR-1206 -> myparts:CAPACITOR-0603
- C14: device myparts:CAPACITOR-0603 -> myparts:CAPACITOR-1206
- C15: device myparts:CAPACITOR-SMD-8 -> myparts:CAPACITOR-0603
- C17: device myparts:CAPACITOR-0603 -> myparts:CAPACITOR-SMD-8
Connections:
- removed net N$7: MOD1.UART1_TX, R10.1, R9.2
- new net N$37: MOD1.UART2_TX, R10.1, R9.2
- net GND: now also C10.1, C26.1, C29.1; no longer C12.1, C28.1, C31.1
- net N$13: now also C21.2, C22.2; no longer C17.2, C18.2
- net N$17: now also C31.1; no longer C29.1
- net N$2: now also C23.2; no longer C21.2
- net N$20: now also D3.K; no longer D4.K
- net N$21: now also C31.2; no longer C29.2
- net N$32: now also C25.2; no longer C23.2
- net N$33: now also D4.K; no longer D5.K
- net N$35: now also C24.2; no longer C22.2
- net N$42: now also C29.2, C30.2; no longer C27.2, C28.2
- net N$49: now also D4.A; no longer D5.A
- net N$50: now also D3.A; no longer D4.A
- net N$57: now also C10.2; no longer C30.2
- net N$6: now also MOD1.UART2_RX; no longer MOD1.UART1_RX
- net N$65: now also C12.2; no longer C11.2
- net N$66: now also C12.1; no longer C11.1
- net N$68: now also C28.2; no longer C26.2
- net N$69: now also C28.1; no longer C26.1
- net N$72: now also C11.1; no longer C10.1
- net N$77: now also C26.2, C27.2; no longer C24.2, C25.2
- net VCC: now also C11.2, C17.2, C18.2; no longer C10.2, C12.2, C31.2
Other:
- moved on the sheet: C10, C11, C12, C13, C14, C16, C18, C19, C20, C21, C22, C23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
