File: eagle/daq.sch (EAGLE design)
At the start: 86 parts

Commit message: fin
Parts:
- removed R29: (no value), myparts:RESISTOR-0805
- removed R30, R31, R32: (no value), myparts:RESISTOR-0603
- added C32, C33, C34, C35: (no value), myparts:CAPACITOR-0603
- R18, R20, R23, R24, R25: device myparts:RESISTOR-0603 -> myparts:RESISTOR-0805
- R21, R22, R26, R28: device myparts:RESISTOR-0805 -> myparts:RESISTOR-0603
Connections:
- removed net N$17: C31.1, IC6.IN-, IC6.VBUS, R27.2
- removed net N$21: C31.2, IC6.IN+, R25.2
- removed net N$68: C28.2, IC5.IN+, R18.1
- removed net N$69: C28.1, IC5.IN-, IC5.VBUS, R20.1
- net GND: now also C29.2, C30.2, C31.1, C32.1, C34.2, C35.2; no longer C29.1, C30.1
- net N$11: now also C28.2, C29.1, IC5.IN+; no longer R21.2
- net N$15: now also R22.2; no longer R24.2
- net N$27: now also R26.2; no longer R30.2
- net N$28: now also R20.1; no longer R22.1
- net N$29: now also R19.1; no longer R21.1
- net N$30: now also R25.1; no longer R29.1
- net N$36: now also R24.1; no longer R28.1
- net N$40: now also C33.2, C34.1, IC6.IN+, R23.2, R24.2; no longer R25.1, R26.2, R28.2
- net N$42: now also C31.2, C32.2; no longer C29.2, C30.2
- net N$5: now also C28.1, C30.1, IC5.IN-, IC5.VBUS, R18.1; no longer R19.1, R22.2
- net N$71: now also R21.2; no longer R23.2
- net N$73: now also R28.2; no longer R32.2
- net N$79: now also R27.2; no longer R31.2
- net N$8: now also C33.1, C35.1, IC6.IN-, IC6.VBUS, R23.1, R25.2; no longer R26.1, R27.1, R29.2
- net VCC: now also R21.1, R22.1, R26.1, R27.1, R28.1; no longer R23.1, R24.1, R30.1, R31.1, R32.1
Other:
- moved on the sheet: C29, C30, C31, R18, R19, R20, R21, R22, R23, R24, R25, R26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
