File: eagle/eagle/daq.brd (EAGLE design)
At the start: 59.7 x 68.6 mm, 86 parts

Commit message: fin
Parts:
- removed D5: (no value), myparts:SOD123-DIODE
- added D3: (no value), myparts:SOD123-DIODE
- C12: device myparts:1206 -> myparts:0603
- C14: device myparts:0603 -> myparts:1206
- C15: device myparts:CAPACITOR-SMD-8 -> myparts:0603
- C17: device myparts:0603 -> myparts:CAPACITOR-SMD-8
- moved C31 43.3 mm to (45.2, 16.1)
- moved C30 31.3 mm to (40.9, 19.3)
- moved C23 24.7 mm to (34.9, 47.2), turned to 180 degrees
- moved C16 24.1 mm to (11.0, 42.7)
- moved C22 21.9 mm to (29.1, 44.2)
- moved C12 17.6 mm to (8.26, 19.4), turned to 270 degrees
- moved C24 14.3 mm to (20.3, 24.1)
- moved C17 11.2 mm to (19.8, 42.5)
- moved C15 8.87 mm to (11.0, 41.1)
- moved C25 8.49 mm to (26.2, 24.1)
- moved C27 7.90 mm to (33.1, 19.3)
- moved D4 6.35 mm to (28.7, 13.1)
- moved C18 6.04 mm to (34.9, 45.7)
- moved C21 6.04 mm to (29.1, 45.7), turned to 0 degrees
- moved C10 5.75 mm to (9.91, 15.2), turned to 0 degrees
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Connections:
- net VEXT renamed N$7
- net GND: now also C10.1, C26.1, C29.1; no longer C12.1, C28.1, C31.1
- net N$13: now also C21.2, C22.2; no longer C17.2, C18.2
- net N$17: now also C31.1; no longer C29.1
- net N$2: now also C23.2; no longer C21.2
- net N$20: now also D3.1; no longer D4.1
- net N$21: now also C31.2; no longer C29.2
- net N$32: now also C25.2; no longer C23.2
- net N$33: now also D4.1; no longer D5.1
- net N$35: now also C24.2; no longer C22.2
- net N$42: now also C29.2, C30.2; no longer C27.2, C28.2
- net N$49: now also D4.2; no longer D5.2
- net N$50: now also D3.2; no longer D4.2
- net N$57: now also C10.2; no longer C30.2
- net N$65: now also C12.2; no longer C11.2
- net N$66: now also C12.1; no longer C11.1
- net N$68: now also C28.2; no longer C26.2
- net N$69: now also C28.1; no longer C26.1
- net N$72: now also C11.1; no longer C10.1
- net N$77: now also C26.2, C27.2; no longer C24.2, C25.2
- net VCC: now also C11.2, C17.2, C18.2; no longer C10.2, C12.2, C31.2
Routing:
- net N$57: vias 2 -> 4
