File: eagle/eagle/daq.sch (EAGLE design)
At the start: 86 parts

Commit message: fin
Parts:
- removed D5: (no value), myparts:DIODE-SCHOTTKY
- added D3: (no value), myparts:DIODE-SCHOTTKY
- C12: device myparts:CAPACITOR-1206 -> myparts:CAPACITOR-0603
- C14: device myparts:CAPACITOR-0603 -> myparts:CAPACITOR-1206
- C15: device myparts:CAPACITOR-SMD-8 -> myparts:CAPACITOR-0603
- C17: device myparts:CAPACITOR-0603 -> myparts:CAPACITOR-SMD-8
Connections:
- net VEXT renamed N$7
- removed net N$7 (its old number): MOD1.UART1_TX, R10.1, R9.2
- new net N$37: MOD1.UART2_TX, R10.1, R9.2
- net GND: now also C10.1, C26.1, C29.1; no longer C12.1, C28.1, C31.1
- net N$13: now also C21.2, C22.2; no longer C17.2, C18.2
- net N$17: now also C31.1; no longer C29.1
- net N$2: now also C23.2; no longer C21.2
- net N$20: now also D3.K; no longer D4.K
- net N$21: now also C31.2; no longer C29.2
- net N$32: now also C25.2; no longer C23.2
- net N$33: now also D4.K; no longer D5.K
- net N$35: now also C24.2; no longer C22.2
- net N$42: now also C29.2, C30.2; no longer C27.2, C28.2
- net N$49: now also D4.A; no longer D5.A
- net N$50: now also D3.A; no longer D4.A
- net N$57: now also C10.2; no longer C30.2
- net N$6: now also MOD1.UART2_RX; no longer MOD1.UART1_RX
- net N$65: now also C12.2; no longer C11.2
- net N$66: now also C12.1; no longer C11.1
- net N$68: now also C28.2; no longer C26.2
- net N$69: now also C28.1; no longer C26.1
- net N$72: now also C11.1; no longer C10.1
- net N$77: now also C26.2, C27.2; no longer C24.2, C25.2
- net VCC: now also C11.2, C17.2, C18.2; no longer C10.2, C12.2, C31.2
Other:
- moved on the sheet: C10, C11, C12, C13, C14, C16, C18, C19, C20, C21, C22, C23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
